Commit message: Add files via upload

File: urdf/assignmentv1.urdf (robot description, URDF)
Before this commit: robot tortoisebot, 30 links, 29 joints
Links:
- link front_caster: geometry collision sphere radius=0.04; visual sphere radius=0.04
- link left_wheel: geometry collision cylinder length=0.02 radius=0.04; visual cylinder length=0.02 radius=0.04
- link rear_caster: geometry collision sphere radius=0.04; visual sphere radius=0.04
- link right_wheel: geometry collision cylinder length=0.02 radius=0.04; visual cylinder length=0.02 radius=0.04
Joints:
- joint front_caster_joint: axis 0 1 0 -> 1 1 1
- joint rear_caster_joint: axis 0 1 0 -> 1 1 1

Commit message: updated .urdf file

File: urdf/assignmentv1.urdf (robot description, URDF)
Before this commit: robot assignment_bot, 30 links, 29 joints
Links:
- link base_link: geometry collision box size=0.6 0.3 0.08; visual mesh filename=package://mcubot/meshes/base.stl scale=1 1 1
